File: newPCB.sch (KiCad schematic (older format))
At the start: 15 parts, among them J1 Conn_01x08_Male, J2 AudioJack3, J3 AudioJack3, SW1 SW_Push_DPDT, U1 TL084

Commit message: Made heirarchical structure, replaced tl084 with tl081, still needs work
Parts:
- removed C3: 260u, Capacitor_THT:CP_Radial_D40.0mm_P10.00mm_3pin_SnapIn, symbol Device:C
- removed C4: 820p, Capacitor_SMD:C_1210_3225Metric_Pad1.42x2.65mm_HandSolder, symbol Device:C
- removed J3: AudioJack3, Connector_Audio:Jack_3.5mm_CUI_SJ-3523-SMT_Horizontal, symbol Connector:AudioJack3
- removed R3: 10k, Resistor_SMD:R_0612_1632Metric_Pad1.18x3.40mm_HandSolder, symbol Device:R
- removed R4: 2.49M, Resistor_SMD:R_0612_1632Metric_Pad1.18x3.40mm_HandSolder, symbol Device:R
- removed RV2: 500k, Potentiometer_THT:Potentiometer_Vishay_148-149_Single_Vertical, symbol Device:R_POT_TRIM
- removed unit 2 of U1
- added C?: 820p, Capacitor_SMD:C_1210_3225Metric_Pad1.42x2.65mm_HandSolder, symbol Device:C
- added C?: 260u, Capacitor_THT:CP_Radial_D40.0mm_P10.00mm_3pin_SnapIn, symbol Device:C
- added C?: C, symbol Device:C
- added R?: 2.49M, Resistor_SMD:R_0612_1632Metric_Pad1.18x3.40mm_HandSolder, symbol Device:R
- added R?: 10k, Resistor_SMD:R_0612_1632Metric_Pad1.18x3.40mm_HandSolder, symbol Device:R
- added RV?: 500k, Potentiometer_THT:Potentiometer_Vishay_148-149_Single_Vertical, symbol Device:R_POT_TRIM
- added U?: TL081, symbol Amplifier_Operational:TL081
Connections:
- net labels added: Amp1_0, GNDS, Node_0, VD, VS
- wire segments 68 -> 66
- no-connect marks 6 -> 8
Other:
- moved on the sheet: C1, C2, J1, J2, R1, R2, RV1, SW1, U1A, U1E

Commit message: Added bypass capacitors to newPCBamps layer, need to implement analog ground in top layer
Parts:
- removed C?: 820p, Capacitor_SMD:C_1210_3225Metric_Pad1.42x2.65mm_HandSolder, symbol Device:C
- removed C?: 260u, Capacitor_THT:CP_Radial_D40.0mm_P10.00mm_3pin_SnapIn, symbol Device:C
- removed C?: C, symbol Device:C
- removed R?: 2.49M, Resistor_SMD:R_0612_1632Metric_Pad1.18x3.40mm_HandSolder, symbol Device:R
- removed R?: 10k, Resistor_SMD:R_0612_1632Metric_Pad1.18x3.40mm_HandSolder, symbol Device:R
- removed RV?: 500k, Potentiometer_THT:Potentiometer_Vishay_148-149_Single_Vertical, symbol Device:R_POT_TRIM
- removed U?: TL081, symbol Amplifier_Operational:TL081
- added C?: 820p, Capacitor_SMD:C_1210_3225Metric_Pad1.42x2.65mm_HandSolder, symbol Device:C
- added C?: 260u, Capacitor_THT:CP_Radial_D40.0mm_P10.00mm_3pin_SnapIn, symbol Device:C
- added C?: C, symbol Device:C
- added R?: 2.49M, Resistor_SMD:R_0612_1632Metric_Pad1.18x3.40mm_HandSolder, symbol Device:R
- added R?: 10k, Resistor_SMD:R_0612_1632Metric_Pad1.18x3.40mm_HandSolder, symbol Device:R
- added RV?: 500k, Potentiometer_THT:Potentiometer_Vishay_148-149_Single_Vertical, symbol Device:R_POT_TRIM
- added U?: TL081, symbol Amplifier_Operational:TL081
Changed lines of the file:
@@
 $Comp
 L power:GNDS #PWR?
-U 1 1 6227322D
+U 1 1 62257E77
 P 2700 6450
 F 0 "#PWR?" H 2700 6200 50  0001 C CNN
@@
 $Comp
 L Device:C C?
-U 1 1 62273235
+U 1 1 62257E78
 P 3850 4850
 F 0 "C?" V 3598 4850 50  0000 C CNN
@@
 $Comp
 L Device:R R?
-U 1 1 6227323B
+U 1 1 62257E79
 P 3850 5250
 F 0 "R?" V 3643 5250 50  0000 C CNN
@@
 $Comp
 L Device:R_POT_TRIM RV?
-U 1 1 62273243
+U 1 1 62257E7A
 P 1700 5250
 F 0 "RV?" V 1493 5250 50  0000 C CNN
@@
 $Comp
 L Device:R R?
-U 1 1 62273249
+U 1 1 62257E7B
 P 2300 5250
 F 0 "R?" V 2093 5250 50  0000 C CNN
@@
 $Comp
 L Device:C C?
-U 1 1 6227324F
+U 1 1 62257E7C
 P 2850 5250
 F 0 "C?" V 2598 5250 50  0000 C CNN
@@
 $Comp
 L Amplifier_Operational:TL081 U?
-U 1 1 6227325A
+U 1 1 62257E7D
 P 3750 6150
 F 0 "U?" H 4094 6196 50  0000 L CNN
@@
 $Comp
 L power:VD #PWR?
-U 1 1 62273268
+U 1 1 62257E7E
 P 3650 6650
 F 0 "#PWR?" H 3650 6500 50  0001 C CNN
@@
 $Comp
 L power:VS #PWR?
-U 1 1 6227326E
+U 1 1 62257E7F
 P 3650 5650
 F 0 "#PWR?" H 3450 5500 50  0001 C CNN
@@
 $Comp
 L power:VS #PWR?
-U 1 1 62273276
+U 1 1 62257E80
 P 1400 6000
 F 0 "#PWR?" H 1200 5850 50  0001 C CNN
@@
 $Comp
 L power:VD #PWR?
-U 1 1 6227327C
+U 1 1 62257E81
 P 1400 6700
 F 0 "#PWR?" H 1400 6550 50  0001 C CNN
@@
 $Comp
 L Device:C C?
-U 1 1 62273282
+U 1 1 62257E82
 P 1400 6350
 F 0 "C?" H 1515 6396 50  0000 L CNN
